Commit message: add tcp

File: urdf/ur5_robotiq_85.urdf (robot description, URDF)
Before this commit: robot ur5_robotiq_85, 20 links, 19 joints
Links:
- added link tcp_link; visual box size=0.01 0.01 0.01
Joints:
- added joint ee_tcp_joint: type fixed, parent ee_link, child tcp_link, origin xyz=0.1 0 0 rpy=0 0 0

Commit message: rotation

File: urdf/ur5_robotiq_85.urdf (robot description, URDF)
Before this commit: robot ur5_robotiq_85, 21 links, 20 joints
Links:
- removed link left_inner_finger
- removed link left_inner_finger_pad
- removed link left_inner_knuckle
- removed link left_outer_finger
- removed link left_outer_knuckle
- removed link right_inner_finger
- removed link right_inner_finger_pad
- removed link right_inner_knuckle
- removed link right_outer_finger
- removed link right_outer_knuckle
- removed link robotiq_arg2f_base_link
Joints:
- removed joint finger_joint
- removed joint left_inner_finger_joint
- removed joint left_inner_finger_pad_joint
- removed joint left_inner_knuckle_joint
- removed joint left_outer_finger_joint
- removed joint right_inner_finger_joint
- removed joint right_inner_finger_pad_joint
- removed joint right_inner_knuckle_joint
- removed joint right_outer_finger_joint
- removed joint right_outer_knuckle_joint
- removed joint robotiq_85_base_joint

Commit message: gripper works

File: urdf/ur5_robotiq_85.urdf (robot description, URDF)
Before this commit: robot ur5_robotiq_85, 10 links, 9 joints
Links:
- added link left_inner_finger, mass 0.0104003125914103; collision mesh filename=../meshes/robotiq_85/collision/robotiq_arg2f_85_inner_finge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 scale=0.001 0.001 0.001; visual mesh filename=../meshes/robotiq_85/visual/robotiq_arg2f_85_inner_finger.d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 scale=0.001 0.001 0.001
- added link left_inner_finger_pad, mass 1.; collision box size=0.022 0.00635 0.0375; visual box size=0.022 0.00635 0.0375
- added link left_inner_knuckle, mass 0.0271177346495152; collision mesh filename=../meshes/robotiq_85/collision/robotiq_arg2f_85_inner_knuck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 scale=0.001 0.001 0.001; visual mesh filename=../meshes/robotiq_85/visual/robotiq_arg2f_85_inner_knuckle.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 scale=0.001 0.001 0.001
- added link left_outer_finger, mass 0.022614240507152; collision mesh filename=../meshes/robotiq_85/collision/robotiq_arg2f_85_outer_finge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 scale=0.001 0.001 0.001; visual mesh filename=../meshes/robotiq_85/visual/robotiq_arg2f_85_outer_finger.d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 scale=0.001 0.001 0.001
- added link left_outer_knuckle, mass 0.00853198276973456; collision mesh filename=../meshes/robotiq_85/collision/robotiq_arg2f_85_outer_knuck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 scale=0.001 0.001 0.001; visual mesh filename=../meshes/robotiq_85/visual/robotiq_arg2f_85_outer_knuckle.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 scale=0.001 0.001 0.001
- added link right_inner_finger, mass 0.0104003125914103; collision mesh filename=../meshes/robotiq_85/collision/robotiq_arg2f_85_inner_finge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 scale=0.001 0.001 0.001; visual mesh filename=../meshes/robotiq_85/visual/robotiq_arg2f_85_inner_finger.d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 scale=0.001 0.001 0.001
- added link right_inner_finger_pad, mass 1; collision box size=0.022 0.00635 0.0375; visual box size=0.022 0.00635 0.0375
- added link right_inner_knuckle, mass 0.0271177346495152; collision mesh filename=../meshes/robotiq_85/collision/robotiq_arg2f_85_inner_knuck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 scale=0.001 0.001 0.001; visual mesh filename=../meshes/robotiq_85/visual/robotiq_arg2f_85_inner_knuckle.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 scale=0.001 0.001 0.001
- added link right_outer_finger, mass 0.022614240507152; collision mesh filename=../meshes/robotiq_85/collision/robotiq_arg2f_85_outer_finge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 scale=0.001 0.001 0.001; visual mesh filename=../meshes/robotiq_85/visual/robotiq_arg2f_85_outer_finger.d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 scale=0.001 0.001 0.001
- added link right_outer_knuckle, mass 0.00853198276973456; collision mesh filename=../meshes/robotiq_85/collision/robotiq_arg2f_85_outer_knuck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 scale=0.001 0.001 0.001; visual mesh filename=../meshes/robotiq_85/visual/robotiq_arg2f_85_outer_knuckle.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 scale=0.001 0.001 0.001
- added link robotiq_arg2f_base_link, mass 0.22652; collision mesh filename=../meshes/robotiq_85/collision/robotiq_arg2f_base_link.stl; visual mesh filename=../meshes/robotiq_85/visual/robotiq_arg2f_85_base_link.dae scale=0.001 0.001 0.001
Joints:
- added joint finger_joint: type revolute, parent robotiq_arg2f_base_link, child left_outer_knuckle, origin xyz=0 -0.0306011 0.054904 rpy=0 0 3.14159265359, axis 1 0 0, limit lower=0 upper=0.8 effort=1000 velocity=2.0
- added joint left_inner_finger_joint: type revolute, parent left_outer_finger, child left_inner_finger, origin xyz=0 0.0061 0.0471 rpy=0 0 0, axis 1 0 0, limit lower=-0.8757 upper=0 effort=1000 velocity=2.0, mimic joint=finger_joint multiplier=-1 offset=0
- added joint left_inner_finger_pad_joint: type fixed, parent left_inner_finger, child left_inner_finger_pad, origin xyz=0 -0.0220203446692936 0.03242 rpy=0 0 0, axis 0 0 1
- added joint left_inner_knuckle_joint: type revolute, parent robotiq_arg2f_base_link, child left_inner_knuckle, origin xyz=0 -0.0127 0.06142 rpy=0 0 3.14159265359, axis 1 0 0, limit lower=0 upper=0.8757 effort=1000 velocity=2.0, mimic joint=finger_joint multiplier=1 offset=0
- added joint left_outer_finger_joint: type fixed, parent left_outer_knuckle, child left_outer_finger, origin xyz=0 0.0315 -0.0041 rpy=0 0 0, axis 1 0 0
- added joint right_inner_finger_joint: type revolute, parent right_outer_finger, child right_inner_finger, origin xyz=0 0.0061 0.0471 rpy=0 0 0, axis 1 0 0, limit lower=-0.8757 upper=0 effort=1000 velocity=2.0, mimic joint=finger_joint multiplier=-1 offset=0
- added joint right_inner_finger_pad_joint: type fixed, parent right_inner_finger, child right_inner_finger_pad, origin xyz=0 -0.0220203446692936 0.03242 rpy=0 0 0, axis 0 0 1
- added joint right_inner_knuckle_joint: type revolute, parent robotiq_arg2f_base_link, child right_inner_knuckle, origin xyz=0 0.0127 0.06142 rpy=0 0 0.0, axis 1 0 0, limit lower=0 upper=0.8757 effort=1000 velocity=2.0, mimic joint=finger_joint multiplier=1 offset=0
- added joint right_outer_finger_joint: type fixed, parent right_outer_knuckle, child right_outer_finger, origin xyz=0 0.0315 -0.0041 rpy=0 0 0, axis 1 0 0
- added joint right_outer_knuckle_joint: type revolute, parent robotiq_arg2f_base_link, child right_outer_knuckle, origin xyz=0 0.0306011 0.054904 rpy=0 0 0, axis 1 0 0, limit lower=0 upper=0.81 effort=1000 velocity=2.0, mimic joint=finger_joint multiplier=1 offset=0
- added joint robotiq_85_base_joint: type fixed, parent ee_link, child robotiq_arg2f_base_link, origin xyz=0 0 0 rpy=0 1.57079632679 0

Commit message: init and load seperated for config in main

File: urdf/ur5_robotiq_85.urdf (robot description, URDF)
Before this commit: robot ur5_robotiq_85, 21 links, 20 joints
Joints:
- joint ee_tcp_joint: origin xyz=0.1 0 0 rpy=0 0 0 -> xyz=0.14 0 0 rpy=0 0 0

Commit message: camera added

File: urdf/ur5_robotiq_85.urdf (robot description, URDF)
Before this commit: robot ur5_robotiq_85, 21 links, 20 joints
Links:
- added link camera_link, mass 0.16; collision mesh filename=../meshes/camera/collision/camera.stl; visual mesh filename=../meshes/camera/visual/camera.obj
Joints:
- added joint ee_camera_joint: type fixed, parent ee_link, child camera_link, origin xyz=0.0 0.0 0.0 rpy=1.57079632679 0.0 1.57079632679
- joint ee_tcp_joint: origin xyz=0.14 0 0 rpy=0 0 0 -> xyz=0.16 0 0 rpy=0 0 0
- joint robotiq_85_base_joint: origin xyz=0 0 0 rpy=0 1.57079632679 0 -> xyz=0.0135 0 0 rpy=0 1.57079632679 0

Commit message: lens added

File: urdf/ur5_robotiq_85.urdf (robot description, URDF)
Before this commit: robot ur5_robotiq_85, 22 links, 21 joints
Links:
- added link lens_link; visual box size=0.005 0.005 0.005
- link tcp_link: geometry visual box size=0.005 0.005 0.005
Joints:
- added joint camera_lens_joint: type fixed, parent camera_link, child lens_link, origin xyz=0 0.042 0.012 rpy=0 -1.04719755119 1.57079632679

Commit message: robotiq camera

File: urdf/ur5_robotiq_85.urdf (robot description, URDF)
Before this commit: robot ur5_robotiq_85, 23 links, 22 joints
Joints:
- joint camera_lens_joint: origin xyz=0 0.042 0.012 rpy=0 -1.04719755119 1.57079632679 -> xyz=0 0.045 0.014 rpy=0 -1.4 1.57079632679

Commit message: removed robotiq camera and reduced resolution to 16x16

File: urdf/ur5_robotiq_85.urdf (robot description, URDF)
Before this commit: robot ur5_robotiq_85, 23 links, 22 joints
Links:
- removed link camera_link
- link tcp_link: geometry 
Joints:
- removed joint camera_lens_joint
- removed joint ee_camera_joint
- added joint ee_lens_joint: type fixed, parent ee_link, child lens_link, origin xyz=0.05 0.0 0.04 rpy=0 0.25 0
- joint ee_tcp_joint: origin xyz=0.16 0 0 rpy=0 0 0 -> xyz=0.14 0 0 rpy=0 0 0
- joint robotiq_85_base_joint: origin xyz=0.0135 0 0 rpy=0 1.57079632679 0 -> xyz=0.0 0 0 rpy=0 1.57079632679 0
